Commit message: fixed small bug in urdf

File: precise_pavp6_support/urdf/pavp6_macro.xacro (robot description, xacro)
@@ -218,5 +218,5 @@
 		<parent link="${prefix}link_5"/>
 		<child link="${prefix}link_6"/>
-		<origin rpy="0.0 0.0 0.0" xyz="0.0 0.0 0.064"/>
+		<origin rpy="0.0 0.0 0.064" xyz="0.0 0.0 0.064"/>
 		<axis xyz="-0.0 0.0 1.000000"/>
 		<!--limit effort="1" lower="-6.283185" upper="6.283185" velocity="1"/-->

Commit message: Revert "fixed small bug in urdf"
This reverts commit 31500cc8881f1cbe4d17ce1cda8c1e4c6ef4f040.

File: precise_pavp6_support/urdf/pavp6_macro.xacro (robot description, xacro)
@@ -218,5 +218,5 @@
 		<parent link="${prefix}link_5"/>
 		<child link="${prefix}link_6"/>
-		<origin rpy="0.0 0.0 0.064" xyz="0.0 0.0 0.064"/>
+		<origin rpy="0.0 0.0 0.0" xyz="0.0 0.0 0.064"/>
 		<axis xyz="-0.0 0.0 1.000000"/>
 		<!--limit effort="1" lower="-6.283185" upper="6.283185" velocity="1"/-->
